Commit message: mesh_integration.urdf file was created to test the urdf build with the cad mesh files, this produced the ideal graph structure and parent/child relations we needed,[ERROR] dae files are out of position and scale

File: src/mob/urdf/mesh_integration.urdf (robot description, URDF)
Before this commit: robot mob_robot, 2 links, 1 joints
Links:
- added link left_ankle, mass 0.0005; collision mesh filename=file:///home/jiovanni/catkin_ws/src/mob/urdf/LeftAnkle.dae scale=0.1, 0.1, 0.1; visual mesh filename=file:///home/jiovanni/catkin_ws/src/mob/urdf/LeftAnkle.dae scale=0.1, 0.1, 0.1
- added link left_arm, mass 0.0005; collision mesh filename=file:///home/jiovanni/catkin_ws/src/mob/urdf/LeftArm.dae scale=0.1, 0.1, 0.1; visual mesh filename=file:///home/jiovanni/catkin_ws/src/mob/urdf/LeftArm.dae scale=0.1, 0.1, 0.1
- added link left_foot, mass 0.0005; collision mesh filename=file:///home/jiovanni/catkin_ws/src/mob/urdf/LeftFoot.dae scale=0.1, 0.1, 0.1; visual mesh filename=file:///home/jiovanni/catkin_ws/src/mob/urdf/LeftFoot.dae scale=0.1, 0.1, 0.1
- added link left_hand, mass 0.0005; collision mesh filename=file:///home/jiovanni/catkin_ws/src/mob/urdf/LeftHand.dae scale=0.1, 0.1, 0.1; visual mesh filename=file:///home/jiovanni/catkin_ws/src/mob/urdf/LeftHand.dae scale=0.1, 0.1, 0.1
- added link left_shin, mass 0.0005; collision mesh filename=file:///home/jiovanni/catkin_ws/src/mob/urdf/Shin.dae scale=0.1, 0.1, 0.1; visual mesh filename=file:///home/jiovanni/catkin_ws/src/mob/urdf/Shin.dae scale=0.1, 0.1, 0.1
- added link left_thigh, mass 0.0005; collision mesh filename=file:///home/jiovanni/catkin_ws/src/mob/urdf/Thigh.dae scale=0.1, 0.1, 0.1; visual mesh filename=file:///home/jiovanni/catkin_ws/src/mob/urdf/Thigh.dae scale=0.1, 0.1, 0.1
- added link right_ankle, mass 0.0005; collision mesh filename=file:///home/jiovanni/catkin_ws/src/mob/urdf/RightAnkle.dae scale=0.1, 0.1, 0.1; visual mesh filename=file:///home/jiovanni/catkin_ws/src/mob/urdf/RightAnkle.dae scale=0.1, 0.1, 0.1
- added link right_arm, mass 0.0005; collision mesh filename=file:///home/jiovanni/catkin_ws/src/mob/urdf/RightArm.dae scale=0.1, 0.1, 0.1; visual mesh filename=file:///home/jiovanni/catkin_ws/src/mob/urdf/RightArm.dae scale=0.1, 0.1, 0.1
- added link right_foot, mass 0.0005; collision mesh filename=file:///home/jiovanni/catkin_ws/src/mob/urdf/RightFoot.dae scale=0.1, 0.1, 0.1; visual mesh filename=file:///home/jiovanni/catkin_ws/src/mob/urdf/RightFoot.dae scale=0.1, 0.1, 0.1
- added link right_hand, mass 0.0005; collision mesh filename=file:///home/jiovanni/catkin_ws/src/mob/urdf/RightHand.dae scale=0.1, 0.1, 0.1; visual mesh filename=file:///home/jiovanni/catkin_ws/src/mob/urdf/RightHand.dae scale=0.1, 0.1, 0.1
- added link right_shin, mass 0.0005; collision mesh filename=file:///home/jiovanni/catkin_ws/src/mob/urdf/Shin.dae scale=0.1, 0.1, 0.1; visual mesh filename=file:///home/jiovanni/catkin_ws/src/mob/urdf/Shin.dae scale=0.1, 0.1, 0.1
- added link right_thigh, mass 0.0005; collision mesh filename=file:///home/jiovanni/catkin_ws/src/mob/urdf/Thigh.dae scale=0.1, 0.1, 0.1; visual mesh filename=file:///home/jiovanni/catkin_ws/src/mob/urdf/Thigh.dae scale=0.1, 0.1, 0.1
- link base_link: geometry collision mesh filename=file:///home/jiovanni/catkin_ws/src/mob/urdf/Chest.dae scale=0.1, 0.1, 0.1; visual mesh filename=file:///home/jiovanni/catkin_ws/src/mob/urdf/Chest.dae scale=0.1, 0.1, 0.1
- link head_motor: geometry collision mesh filename=file:///home/jiovanni/catkin_ws/src/mob/urdf/HeadMotor.dae scale=0.004, 0.004, 0.004; visual mesh filename=file:///home/jiovanni/catkin_ws/src/mob/urdf/HeadMotor.dae scale=0.004, 0.004, 0.004
Joints:
- added joint Right_shin_joint: type revolute, parent right_thigh, child right_shin, origin xyz=0 0 0 rpy=0 0 0, axis 0 0 1, limit lower=-1.0 upper=1.0 effort=1000.0 velocity=0.5
- added joint left_ankle_joint: type revolute, parent left_shin, child left_ankle, origin xyz=0 0 0 rpy=0 0 0, axis 0 0 1, limit lower=-1.0 upper=1.0 effort=1000.0 velocity=0.5
- added joint left_arm_joint: type revolute, parent base_link, child left_arm, origin xyz=0 0 0 rpy=0 0 0, axis 0 0 1, limit lower=-1.0 upper=1.0 effort=1000.0 velocity=0.5
- added joint left_foot_joint: type revolute, parent left_ankle, child left_foot, origin xyz=0 0 0 rpy=0 0 0, axis 0 0 1, limit lower=-1.0 upper=1.0 effort=1000.0 velocity=0.5
- added joint left_hand_joint: type revolute, parent left_arm, child left_hand, origin xyz=0 0 0 rpy=0 0 0, axis 0 0 1, limit lower=-1.0 upper=1.0 effort=1000.0 velocity=0.5
- added joint left_shin_joint: type revolute, parent left_thigh, child left_shin, origin xyz=0 0 0 rpy=0 0 0, axis 0 0 1, limit lower=-1.0 upper=1.0 effort=1000.0 velocity=0.5
- added joint left_thigh_joint: type revolute, parent base_link, child left_thigh, origin xyz=0 0 0 rpy=0 0 0, axis 0 0 1, limit lower=-1.0 upper=1.0 effort=1000.0 velocity=0.5
- added joint right_ankle_joint: type revolute, parent right_shin, child right_ankle, origin xyz=0 0 0 rpy=0 0 0, axis 0 0 1, limit lower=-1.0 upper=1.0 effort=1000.0 velocity=0.5
- added joint right_arm_joint: type revolute, parent base_link, child right_arm, origin xyz=0 0 0 rpy=0 0 0, axis 0 0 1, limit lower=-1.0 upper=1.0 effort=1000.0 velocity=0.5
- added joint right_foot_joint: type revolute, parent right_ankle, child right_foot, origin xyz=0 0 0 rpy=0 0 0, axis 0 0 1, limit lower=-1.0 upper=1.0 effort=1000.0 velocity=0.5
- added joint right_hand_joint: type revolute, parent right_arm, child right_hand, origin xyz=0 0 0 rpy=0 0 0, axis 0 0 1, limit lower=-1.0 upper=1.0 effort=1000.0 velocity=0.5
- added joint right_thigh_joint: type revolute, parent base_link, child right_thigh, origin xyz=0 0 0 rpy=0 0 0, axis 0 0 1, limit lower=-1.0 upper=1.0 effort=1000.0 velocity=0.5
- joint head_joint: origin xyz=0 0 0.07 rpy=0 0 0 -> xyz=0 0 0 rpy=0 0 0
