Commit message: Worked on experimental body

File: src/mob/urdf/mob_experimental_build.urdf (robot description, URDF)
Before this commit: robot mob_robot, 2 links, 1 joints
Links:
- added link left_ankle_link, mass 0.055; collision box size=0.0407 0.0197 0.0429; collision box size=0.0435 0.0252 0.05588
- added link left_foot_link, mass 0.055; collision box size=0.0407 0.0197 0.0429; collision box size=0.125 0.062 0.002
- added link left_hip_link, mass 0.055; collision box size=0.025 0.055 0.065; collision box size=0.056 0.025 0.044
- added link left_knee_link, mass 0.055; collision box size=0.0285 0.0433 0.1; visual box size=0.0256 0.0563 0.0874
- added link left_shoulder, mass 0.055; collision box size=0.055 0.044 0.04; visual box size=0.055 0.044 0.04
- added link left_thigh_link, mass 0.055; collision box size=0.0285 0.0433 0.1; visual box size=0.0285 0.0433 0.1
- added link right_ankle_link, mass 0.055; collision box size=0.0407 0.0197 0.0429; collision box size=0.0435 0.0252 0.05588
- added link right_arm_link, mass 0.055; collision box size=0.025 0.055 0.065; collision box size=0.407 0.197 0.429
- added link right_foot_link, mass 0.055; collision box size=0.0407 0.0197 0.0429; collision box size=0.125 0.062 0.002
- added link right_hip_link, mass 0.055; collision box size=0.025 0.055 0.065; collision box size=0.056 0.025 0.044
- added link right_knee_link, mass 0.055; collision box size=0.0285 0.0433 0.1; visual box size=0.0256 0.0563 0.0874
- added link right_shoulder, mass 0.055; collision box size=0.055 0.044 0.04; visual box size=0.055 0.044 0.04
- added link right_thigh_link, mass 0.055; collision box size=0.0285 0.0433 0.1; visual box size=0.0285 0.0433 0.1
- link base_link: geometry collision box size=0.02905 0.09013 0.04335; collision box size=0.407 0.197 0.429
Joints:
- added joint left_ankle_joint_roll: type revolute, parent left_ankle_link, child left_foot_link, origin xyz=0 0 -0.05 rpy=0 0 0, axis 1 0 0, limit lower=-1.0 upper=1.0 effort=1000.0 velocity=0.5
- added joint left_hip_joint_pitch: type revolute, parent left_hip_link, child left_thigh_link, origin xyz=0 0 -0.07 rpy=0 0 0, axis 0 1 0, limit lower=-1.0 upper=1.0 effort=1000.0 velocity=0.5
- added joint left_hip_joint_roll: type revolute, parent base_link, child left_hip_link, origin xyz=0 -0.03 -0.0245 rpy=0 0 0, axis 1 0 0, limit lower=-1.0 upper=1.0 effort=1000.0 velocity=0.5
- added joint left_knee_joint_pitch: type revolute, parent left_knee_link, child left_ankle_link, origin xyz=0 0 -0.075 rpy=0 0 0, axis 0 1 0, limit lower=-1.0 upper=1.0 effort=1000.0 velocity=0.5
- added joint left_shoulder_joint: type revolute, parent base_link, child left_shoulder, origin xyz=0 -0.06 0.045 rpy=0 0 0, axis 0 1 0, limit lower=-1.0 upper=1.0 effort=1000.0 velocity=0.5
- added joint left_thigh_joint_pitch: type revolute, parent left_thigh_link, child left_knee_link, origin xyz=0 0 -0.10 rpy=0 0 0, axis 0 1 0, limit lower=-1.0 upper=1.0 effort=1000.0 velocity=0.5
- added joint right_ankle_joint_roll: type revolute, parent right_ankle_link, child right_foot_link, origin xyz=0 0 -0.05 rpy=0 0 0, axis 1 0 0, limit lower=-1.0 upper=1.0 effort=1000.0 velocity=0.5
- added joint right_arm_joint: type revolute, parent right_shoulder, child right_arm_link, origin xyz=0 0 0 rpy=0 0 0, axis 1 0 0, limit lower=-1.0 upper=1.0 effort=1000.0 velocity=0.5
- added joint right_hip_joint_pitch: type revolute, parent right_hip_link, child right_thigh_link, origin xyz=0 0 -0.07 rpy=0 0 0, axis 0 1 0, limit lower=-1.0 upper=1.0 effort=1000.0 velocity=0.5
- added joint right_hip_joint_roll: type revolute, parent base_link, child right_hip_link, origin xyz=0 0.03 -0.0245 rpy=0 0 0, axis 1 0 0, limit lower=-1.0 upper=1.0 effort=1000.0 velocity=0.5
- added joint right_knee_joint_pitch: type revolute, parent right_knee_link, child right_ankle_link, origin xyz=0 0 -0.075 rpy=0 0 0, axis 0 1 0, limit lower=-1.0 upper=1.0 effort=1000.0 velocity=0.5
- added joint right_shoulder_joint: type revolute, parent base_link, child right_shoulder, origin xyz=0 0.06 0.045 rpy=0 0 0, axis 0 1 0, limit lower=-1.0 upper=1.0 effort=1000.0 velocity=0.5
- added joint right_thigh_joint_pitch: type revolute, parent right_thigh_link, child right_knee_link, origin xyz=0 0 -0.10 rpy=0 0 0, axis 0 1 0, limit lower=-1.0 upper=1.0 effort=1000.0 velocity=0.5
- joint head_joint: origin xyz=0 0 0.07 rpy=0 0 0 -> xyz=0 0 0.079 rpy=0 0 0

Commit message: MOB full

File: src/mob/urdf/mob_experimental_build.urdf (robot description, URDF)
Before this commit: robot mob_robot, 15 links, 14 joints
Links:
- added link left_arm_link, mass 0.055; collision box size=0.025 0.055 0.065; collision box size=0.407 0.197 0.429
- added link left_hand, mass 0.055; collision box size=0.407 0.197 0.429; visual box size=0.0407 0.0197 0.0429
- added link right_hand, mass 0.055; collision box size=0.407 0.197 0.429; visual box size=0.0407 0.0197 0.0429
Joints:
- added joint left_arm_joint: type revolute, parent left_shoulder, child left_arm_link, origin xyz=0 -0.022 0.02 rpy=0 0 0, axis 1 0 0, limit lower=-1.0 upper=1.0 effort=1000.0 velocity=0.5
- added joint left_hand_joint: type revolute, parent left_arm_link, child left_hand, origin xyz=0 0 -0.085 rpy=0 0 0, axis 1 0 0, limit lower=-1.0 upper=1.0 effort=1000.0 velocity=0.5
- added joint right_hand_joint: type revolute, parent right_arm_link, child right_hand, origin xyz=0 0 -0.085 rpy=0 0 0, axis 1 0 0, limit lower=-1.0 upper=1.0 effort=1000.0 velocity=0.5
- joint right_arm_joint: origin xyz=0 0 0 rpy=0 0 0 -> xyz=0 0.022 0.02 rpy=0 0 0
