Commit message: created robot foot in urdf

File: src/mob/urdf/mob_robot.urdf (robot description, URDF)
Before this commit: robot mob_robot, 1 links, 0 joints
Links:
- link base_link: mass None -> 2; geometry collision box size=0.125 0.062 0.02; visual box size=0.125 0.062 0.02

Commit message: changed the name with in the urdf now base link is left_foot

File: src/mob/urdf/mob_robot.urdf (robot description, URDF)
Before this commit: robot mob_robot, 1 links, 0 joints
Links:
- removed link base_link
- added link left_foot, mass 2; collision box size=0.125 0.062 0.02; visual box size=0.125 0.062 0.02

Commit message: Base Link name cannot be changed otherwise rviz will load the model in error state

File: src/mob/urdf/mob_robot.urdf (robot description, URDF)
Before this commit: robot mob_robot, 1 links, 0 joints
Links:
- removed link left_foot
- added link base_link, mass 2; collision box size=0.125 0.062 0.02; visual box size=0.125 0.062 0.02

Commit message: Finished left food with attached motor

File: src/mob/urdf/mob_robot.urdf (robot description, URDF)
Before this commit: robot mob_robot, 1 links, 0 joints
Links:
- added link left_foot_motor, mass 0.055; collision box size=0.407 0.197 0.429; visual box size=0.0407 0.0197 0.0429
- link base_link: mass 2 -> 0.0005
Joints:
- added joint left_foot_joint: type fixed, parent base_link, child left_foot_motor, origin xyz=0 0 0.01 rpy=0 0 0, axis 0 0 0.01

Commit message: left leg

File: src/mob/urdf/mob_robot.urdf (robot description, URDF)
Before this commit: robot mob_robot, 2 links, 1 joints
Links:
- removed link left_foot_motor
- added link ankle_link; visual box size=0.0407 0.0197 0.0429; visual box size=0.0435 0.0252 0.05588
- added link hip_link; visual box size=0.025 0.055 0.065; visual box size=0.056 0.025 0.044
- added link hip_motor_link; visual box size=0.0407 0.0197 0.0429
- added link knee_link; visual box size=0.0256 0.0563 0.0874
- added link thigh_link; visual box size=0.0285 0.0433 0.1
- link base_link: mass 0.0005 -> None; geometry visual box size=0.0407 0.0197 0.0429; visual box size=0.125 0.062 0.002
Joints:
- removed joint left_foot_joint
- added joint ankle_joint_roll: type revolute, parent base_link, child ankle_link, origin xyz=0 0 0.014 rpy=0 0 0, axis 1 0 0, limit lower=-1.0 upper=1.0 effort=1000.0 velocity=0.5
- added joint hip_joint_pitch: type revolute, parent thigh_link, child hip_link, origin xyz=0 0 0.07 rpy=0 0 0, axis 0 1 0, limit lower=-1.0 upper=1.0 effort=1000.0 velocity=0.5
- added joint hip_joint_roll: type revolute, parent hip_link, child hip_motor_link, origin xyz=0 0 0.07 rpy=0 0 0, axis 1 0 0, limit lower=-1.0 upper=1.0 effort=1000.0 velocity=0.5
- added joint knee_joint_pitch: type revolute, parent ankle_link, child knee_link, origin xyz=0 0 0.045 rpy=0 0 0, axis 0 1 0, limit lower=-1.0 upper=1.0 effort=1000.0 velocity=0.5
- added joint thigh_joint_pitch: type revolute, parent knee_link, child thigh_link, origin xyz=0 0 0.06 rpy=0 0 0, axis 0 1 0, limit lower=-1.0 upper=1.0 effort=1000.0 velocity=0.5

Commit message: The two legs

File: src/mob/urdf/mob_robot.urdf (robot description, URDF)
Before this commit: robot mob_robot, 6 links, 5 joints
Links:
- removed link ankle_link
- removed link hip_link
- removed link hip_motor_link
- removed link knee_link
- removed link thigh_link
- added link left_ankle_link; visual box size=0.0407 0.0197 0.0429; visual box size=0.0435 0.0252 0.05588
- added link left_hip_link; visual box size=0.025 0.055 0.065; visual box size=0.056 0.025 0.044
- added link left_hip_motor_link; visual box size=0.0407 0.0197 0.0429
- added link left_knee_link; visual box size=0.0256 0.0563 0.0874
- added link left_thigh_link; visual box size=0.0285 0.0433 0.1
- added link right_ankle_link; visual box size=0.0407 0.0197 0.0429; visual box size=0.0435 0.0252 0.05588
- added link right_hip_link; visual box size=0.025 0.055 0.065; visual box size=0.056 0.025 0.044
- added link right_hip_motor_link; visual box size=0.0407 0.0197 0.0429
- added link right_knee_link; visual box size=0.0256 0.0563 0.0874
- added link right_thigh_link; visual box size=0.0285 0.0433 0.1
- link base_link: geometry visual box size=0.0407 0.0197 0.0429; visual box size=0.0407 0.0197 0.0429
Joints:
- removed joint ankle_joint_roll
- removed joint hip_joint_pitch
- removed joint hip_joint_roll
- removed joint knee_joint_pitch
- removed joint thigh_joint_pitch
- added joint left_ankle_joint_roll: type revolute, parent base_link, child left_ankle_link, origin xyz=0 0 0.014 rpy=0 0 0, axis 1 0 0, limit lower=-1.0 upper=1.0 effort=1000.0 velocity=0.5
- added joint left_hip_joint_pitch: type revolute, parent left_thigh_link, child left_hip_link, origin xyz=0 0 0.07 rpy=0 0 0, axis 0 1 0, limit lower=-1.0 upper=1.0 effort=1000.0 velocity=0.5
- added joint left_hip_joint_roll: type revolute, parent left_hip_link, child left_hip_motor_link, origin xyz=0 0 0.07 rpy=0 0 0, axis 1 0 0, limit lower=-1.0 upper=1.0 effort=1000.0 velocity=0.5
- added joint left_knee_joint_pitch: type revolute, parent left_ankle_link, child left_knee_link, origin xyz=0 0 0.045 rpy=0 0 0, axis 0 1 0, limit lower=-1.0 upper=1.0 effort=1000.0 velocity=0.5
- added joint left_thigh_joint_pitch: type revolute, parent left_knee_link, child left_thigh_link, origin xyz=0 0 0.06 rpy=0 0 0, axis 0 1 0, limit lower=-1.0 upper=1.0 effort=1000.0 velocity=0.5
- added joint right_ankle_joint_roll: type revolute, parent base_link, child right_ankle_link, origin xyz=0 0.08 0.014 rpy=0 0 0, axis 1 0 0, limit lower=-1.0 upper=1.0 effort=1000.0 velocity=0.5
- added joint right_hip_joint_pitch: type revolute, parent right_thigh_link, child right_hip_link, origin xyz=0 0 0.07 rpy=0 0 0, axis 0 1 0, limit lower=-1.0 upper=1.0 effort=1000.0 velocity=0.5
- added joint right_hip_joint_roll: type revolute, parent right_hip_link, child right_hip_motor_link, origin xyz=0 0 0.07 rpy=0 0 0, axis 1 0 0, limit lower=-1.0 upper=1.0 effort=1000.0 velocity=0.5
- added joint right_knee_joint_pitch: type revolute, parent right_ankle_link, child right_knee_link, origin xyz=0 0 0.045 rpy=0 0 0, axis 0 1 0, limit lower=-1.0 upper=1.0 effort=1000.0 velocity=0.5
- added joint right_thigh_joint_pitch: type revolute, parent right_knee_link, child right_thigh_link, origin xyz=0 0 0.06 rpy=0 0 0, axis 0 1 0, limit lower=-1.0 upper=1.0 effort=1000.0 velocity=0.5

Commit message: Added Physics, created xacro version of urdf, added a gazebo file for friction coefficients, created material xacro for keeping the color grey in gazebo. Fixed gazebo bug and now robot can be loaded into sim

File: src/mob/urdf/mob_robot.urdf (robot description, URDF)
Before this commit: robot mob_robot, 18 links, 17 joints
Links:
- link base_link: mass 0.0005 -> 0.3445
- link head_motor: mass 0.0005 -> 0.055
- link left_ankle: mass 0.0005 -> 0.0879
- link left_arm: mass 0.0005 -> 0.0919
- link left_foot: mass 0.0005 -> 0.1058
- link left_hand: mass 0.0005 -> 0.0766
- link left_knee: mass 0.0005 -> 0.14
- link left_shin: mass 0.0005 -> 0.0219
- link left_shoulder: mass 0.0005 -> 0.0179
- link left_thigh: mass 0.0005 -> 0.0219
- link right_ankle: mass 0.0005 -> 0.0.0879
- link right_arm: mass 0.0005 -> 0.0919
- link right_foot: mass 0.0005 -> 0.1058
- link right_hand: mass 0.0005 -> 0.0766
- link right_knee: mass 0.0005 -> 0.14
- link right_shin: mass 0.0005 -> 0.0219
- link right_shoulder: mass 0.0005 -> 0.0179
- link right_thigh: mass 0.0005 -> 0.0219
