Commit message: Gazebo working

File: src/mob/urdf/robot_backup.xacro (robot description, xacro)
@@ -29,5 +29,5 @@
     <inertial>
       <mass value="0.3445"/>
-      <inertia ixx="0.1" ixy="0.0" ixz="0.0" iyy="0.1" iyz="0.0" izz="0.1" />
+      <inertia ixx="0.0002431" ixy="0.0" ixz="0.0" iyy="0.00038005" iyz="0.0" izz="0.00022233" />
     </inertial>
   </link>
@@ -59,5 +59,5 @@
     <inertial>
       <mass value="0.055"/>
-      <inertia ixx="0.1" ixy="0.0" ixz="0.0" iyy="0.1" iyz="0.0" izz="0.1" />
+      <inertia ixx="0.0002431" ixy="0.0" ixz="0.0" iyy="0.00038005" iyz="0.0" izz="0.00022233" />
     </inertial>
   </link>
@@ -89,5 +89,5 @@
     <inertial>
       <mass value="0.0179"/>
-      <inertia ixx="0.1" ixy="0.0" ixz="0.0" iyy="0.1" iyz="0.0" izz="0.1" />
+      <inertia ixx="0.0002431" ixy="0.0" ixz="0.0" iyy="0.00038005" iyz="0.0" izz="0.00022233" />
     </inertial>
   </link>
@@ -119,5 +119,5 @@
     <inertial>
       <mass value="0.0919"/>
-      <inertia ixx="0.1" ixy="0.0" ixz="0.0" iyy="0.1" iyz="0.0" izz="0.1" />
+      <inertia ixx="0.0002431" ixy="0.0" ixz="0.0" iyy="0.00038005" iyz="0.0" izz="0.00022233" />
     </inertial>
   </link>
@@ -149,5 +149,5 @@
     <inertial>
       <mass value="0.0766"/>
-      <inertia ixx="0.1" ixy="0.0" ixz="0.0" iyy="0.1" iyz="0.0" izz="0.1" />
+      <inertia ixx="0.0002431" ixy="0.0" ixz="0.0" iyy="0.00038005" iyz="0.0" izz="0.00022233" />
     </inertial>
   </link>
@@ -179,5 +179,5 @@
     <inertial>
       <mass value="0.0219"/>
-      <inertia ixx="0.1" ixy="0.0" ixz="0.0" iyy="0.1" iyz="0.0" izz="0.1" />
+      <inertia ixx="0.0002431" ixy="0.0" ixz="0.0" iyy="0.00038005" iyz="0.0" izz="0.00022233" />
     </inertial>
   </link>
@@ -209,5 +209,5 @@
     <inertial>
       <mass value="0.14"/>
-      <inertia ixx="0.1" ixy="0.0" ixz="0.0" iyy="0.1" iyz="0.0" izz="0.1" />
+      <inertia ixx="0.0002431" ixy="0.0" ixz="0.0" iyy="0.00038005" iyz="0.0" izz="0.00022233" />
     </inertial>
   </link>
@@ -239,5 +239,5 @@
     <inertial>
       <mass value="0.0219"/>
-      <inertia ixx="0.1" ixy="0.0" ixz="0.0" iyy="0.1" iyz="0.0" izz="0.1" />
+      <inertia ixx="0.0002431" ixy="0.0" ixz="0.0" iyy="0.00038005" iyz="0.0" izz="0.00022233" />
     </inertial>
   </link>
@@ -269,5 +269,5 @@
     <inertial>
       <mass value="0.0.0879"/>
-      <inertia ixx="0.1" ixy="0.0" ixz="0.0" iyy="0.1" iyz="0.0" izz="0.1" />
+      <inertia ixx="0.0002431" ixy="0.0" ixz="0.0" iyy="0.00038005" iyz="0.0" izz="0.00022233" />
     </inertial>
   </link>
@@ -299,5 +299,5 @@
     <inertial>
       <mass value="0.1058"/>
-      <inertia ixx="0.1" ixy="0.0" ixz="0.0" iyy="0.1" iyz="0.0" izz="0.1" />
+      <inertia ixx="0.0002431" ixy="0.0" ixz="0.0" iyy="0.00038005" iyz="0.0" izz="0.00022233" />
     </inertial>
   </link>
@@ -329,5 +329,5 @@
     <inertial>
       <mass value="0.0179"/>
-      <inertia ixx="0.1" ixy="0.0" ixz="0.0" iyy="0.1" iyz="0.0" izz="0.1" />
+      <inertia ixx="0.0002431" ixy="0.0" ixz="0.0" iyy="0.00038005" iyz="0.0" izz="0.00022233" />
     </inertial>
   </link>
@@ -359,5 +359,5 @@
     <inertial>
       <mass value="0.0919"/>
-      <inertia ixx="0.1" ixy="0.0" ixz="0.0" iyy="0.1" iyz="0.0" izz="0.1" />
+      <inertia ixx="0.0002431" ixy="0.0" ixz="0.0" iyy="0.00038005" iyz="0.0" izz="0.00022233" />
     </inertial>
   </link>
@@ -389,5 +389,5 @@
     <inertial>
       <mass value="0.0766"/>
-      <inertia ixx="0.1" ixy="0.0" ixz="0.0" iyy="0.1" iyz="0.0" izz="0.1" />
+      <inertia ixx="0.0002431" ixy="0.0" ixz="0.0" iyy="0.00038005" iyz="0.0" izz="0.00022233" />
     </inertial>
   </link>
@@ -419,5 +419,5 @@
     <inertial>
       <mass value="0.0219"/>
-      <inertia ixx="0.1" ixy="0.0" ixz="0.0" iyy="0.1" iyz="0.0" izz="0.1" />
+      <inertia ixx="0.0002431" ixy="0.0" ixz="0.0" iyy="0.00038005" iyz="0.0" izz="0.00022233" />
     </inertial>
   </link>
@@ -449,5 +449,5 @@
     <inertial>
       <mass value="0.14"/>
-      <inertia ixx="0.1" ixy="0.0" ixz="0.0" iyy="0.1" iyz="0.0" izz="0.1" />
+      <inertia ixx="0.0002431" ixy="0.0" ixz="0.0" iyy="0.00038005" iyz="0.0" izz="0.00022233" />
     </inertial>
   </link>
@@ -479,5 +479,5 @@
     <inertial>
       <mass value="0.0219"/>
-      <inertia ixx="0.1" ixy="0.0" ixz="0.0" iyy="0.1" iyz="0.0" izz="0.1" />
+      <inertia ixx="0.0002431" ixy="0.0" ixz="0.0" iyy="0.00038005" iyz="0.0" izz="0.00022233" />
     </inertial>
   </link>
@@ -509,5 +509,5 @@
     <inertial>
       <mass value="0.0879"/>
-      <inertia ixx="0.1" ixy="0.0" ixz="0.0" iyy="0.1" iyz="0.0" izz="0.1" />
+      <inertia ixx="0.0002431" ixy="0.0" ixz="0.0" iyy="0.00038005" iyz="0.0" izz="0.00022233" />
     </inertial>
   </link>
@@ -539,5 +539,5 @@
     <inertial>
       <mass value="0.1058"/>
-      <inertia ixx="0.1" ixy="0.0" ixz="0.0" iyy="0.1" iyz="0.0" izz="0.1" />
+      <inertia ixx="0.0002431" ixy="0.0" ixz="0.0" iyy="0.00038005" iyz="0.0" izz="0.00022233" />
     </inertial>
   </link>
